Commit message: 1

File: torch_robotics/data/urdf/robots/franka_description/robots/panda_arm_no_gripper.urdf (robot description, URDF)
Before this commit: robot panda, 11 links, 10 joints
Joints:
- joint panda_joint1: limit lower=-2.8973 upper=2.8973 effort=87 velocity=2.1750 -> lower=-4.8973 upper=4.8973 effort=87 velocity=2.1750
- joint panda_joint2: limit lower=-1.7628 upper=1.7628 effort=87 velocity=2.1750 -> lower=-3.7628 upper=3.7628 effort=87 velocity=2.1750
- joint panda_joint3: limit lower=-2.8973 upper=2.8973 effort=87 velocity=2.1750 -> lower=-4.8973 upper=4.8973 effort=87 velocity=2.1750
- joint panda_joint4: limit lower=-3.0718 upper=-0.0698 effort=87 velocity=2.1750 -> lower=-3.0718 upper=2.0698 effort=87 velocity=2.1750
- joint panda_joint5: limit lower=-2.8973 upper=2.8973 effort=12 velocity=2.6100 -> lower=-4.8973 upper=4.8973 effort=12 velocity=2.6100
- joint panda_joint6: limit lower=-0.0175 upper=3.7525 effort=12 velocity=2.6100 -> lower=-2.0175 upper=3.7525 effort=12 velocity=2.6100
- joint panda_joint7: limit lower=-2.8973 upper=2.8973 effort=12 velocity=2.6100 -> lower=-3.8973 upper=3.8973 effort=12 velocity=2.6100

Commit message: 3.11修改优化器-有轨迹

File: torch_robotics/data/urdf/robots/franka_description/robots/panda_arm_no_gripper.urdf (robot description, URDF)
Before this commit: robot panda, 11 links, 10 joints
Joints:
- joint panda_joint1: limit lower=-4.8973 upper=4.8973 effort=87 velocity=2.1750 -> lower=-2.8973 upper=2.8973 effort=87 velocity=2.1750
- joint panda_joint2: limit lower=-3.7628 upper=3.7628 effort=87 velocity=2.1750 -> lower=-1.7628 upper=1.7628 effort=87 velocity=2.1750
- joint panda_joint3: limit lower=-4.8973 upper=4.8973 effort=87 velocity=2.1750 -> lower=-2.8973 upper=2.8973 effort=87 velocity=2.1750
- joint panda_joint4: limit lower=-3.0718 upper=2.0698 effort=87 velocity=2.1750 -> lower=-3.0718 upper=-0.0698 effort=87 velocity=2.1750
- joint panda_joint5: limit lower=-4.8973 upper=4.8973 effort=12 velocity=2.6100 -> lower=-2.8973 upper=2.8973 effort=12 velocity=2.6100
- joint panda_joint6: limit lower=-2.0175 upper=3.7525 effort=12 velocity=2.6100 -> lower=-0.0175 upper=3.7525 effort=12 velocity=2.6100
- joint panda_joint7: limit lower=-3.8973 upper=3.8973 effort=12 velocity=2.6100 -> lower=-2.8973 upper=2.8973 effort=12 velocity=2.6100
