Commit message: 5.6

File: torch_robotics/data/urdf/robots/franka_panda_car/robots/franka_panda.urdf (robot description, URDF)
Before this commit: robot panda, 11 links, 10 joints
Links:
- link base_link: mass 5.0 -> None
- link panda_hand: geometry collision mesh filename=package://home/ylc/mpd-public/deps/torch_robotics/torch_rob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; visual mesh filename=package://home/ylc/mpd-public/deps/torch_robotics/torch_rob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
- link panda_link0: geometry collision mesh filename=package://home/ylc/mpd-public/deps/torch_robotics/torch_rob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; visual mesh filename=package://home/ylc/mpd-public/deps/torch_robotics/torch_rob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
- link panda_link1: geometry collision mesh filename=package://home/ylc/mpd-public/deps/torch_robotics/torch_rob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; visual mesh filename=package://home/ylc/mpd-public/deps/torch_robotics/torch_rob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
- link panda_link2: geometry collision mesh filename=package://home/ylc/mpd-public/deps/torch_robotics/torch_rob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; visual mesh filename=package://home/ylc/mpd-public/deps/torch_robotics/torch_rob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
- link panda_link3: geometry collision mesh filename=package://home/ylc/mpd-public/deps/torch_robotics/torch_rob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; visual mesh filename=package://home/ylc/mpd-public/deps/torch_robotics/torch_rob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
- link panda_link4: geometry collision mesh filename=package://home/ylc/mpd-public/deps/torch_robotics/torch_rob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; visual mesh filename=package://home/ylc/mpd-public/deps/torch_robotics/torch_rob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
- link panda_link5: geometry collision mesh filename=package://home/ylc/mpd-public/deps/torch_robotics/torch_rob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; visual mesh filename=package://home/ylc/mpd-public/deps/torch_robotics/torch_rob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
- link panda_link6: geometry collision mesh filename=package://home/ylc/mpd-public/deps/torch_robotics/torch_rob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; visual mesh filename=package://home/ylc/mpd-public/deps/torch_robotics/torch_rob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
- link panda_link7: geometry collision mesh filename=package://home/ylc/mpd-public/deps/torch_robotics/torch_rob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; visual mesh filename=package://home/ylc/mpd-public/deps/torch_robotics/torch_rob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
